Commit message: Add tuned SLAM params, localization mode, map saving, RViz config, and proper URDF
- slam_rtabmap_lidar3d.launch.py: add outdoor-tuned ICP/RTAB-Map parameters
  (point-to-plane ICP, F2M odometry, proximity loop closure, Nav2-ready grid),
  robot_state_publisher from URDF, database_path + rviz launch args
- urdf/amiga_min.urdf: expand to full geometry with visual/collision/inertia
  for base_link (ground-level center) and velodyne (estimated z=0.80 m mount)
- tf_static_base_to_velodyne.launch.py: update z from 0 → 0.80 m to match URDF
- slam_localization.launch.py: new launch file; runs RTAB-Map with
  Mem/IncrementalMemory=false to localise against a saved database without
  extending the map
- slam_bag_replay.launch.py: pass database_path arg through to SLAM stack
- rviz/slam_lidar.rviz: new RViz2 config showing TF, live cloud, map cloud,
  2-D occupancy map, ICP odometry, SLAM trajectory, and robot model
- scripts/save_map.sh: copy rtabmap.db to timestamped directory, generate
  a ready-to-run localise.sh for the saved map
- CLAUDE.md: document all new commands and pending calibration details

https://claude.ai/code/session_01L5i6Nt8m6M2g1D91Wvos4e

File: src/amiga_bringup/urdf/amiga_min.urdf (robot description, URDF)
Before this commit: robot amiga_min, 2 links, 1 joints
Links:
- link base_link: mass None -> 75.0; geometry collision box size=1.10 0.93 0.76; visual box size=1.10 0.93 0.76
- link velodyne: mass None -> 0.83; geometry collision cylinder length=0.072 radius=0.052; visual cylinder length=0.072 radius=0.052
Joints:
- joint base_to_velodyne: origin xyz=0 0 0 rpy=0 0 0 -> xyz=0.0 0.0 0.80 rpy=0 0 0

Commit message: Set physical LiDAR mount calibration: x=1.130 m, y=0, z=0.80 m
Measured 2025-03-05 on the physical Amiga robot:
  x = 1.130 m (44.5 in) — wheelbase midpoint to VLP-16 spin axis, forward
  y = 0.000 m            — centered on robot centreline
  z = 0.800 m            — LiDAR spin axis height above ground
  roll = pitch = yaw = 0 — mount is level, LiDAR front aligns with robot +x

Updated in both:
  - launch/tf_static_base_to_velodyne.launch.py (--x arg)
  - urdf/amiga_min.urdf (base_to_velodyne joint origin)
  - CLAUDE.md (calibration section marked complete)

https://claude.ai/code/session_01L5i6Nt8m6M2g1D91Wvos4e

File: src/amiga_bringup/urdf/amiga_min.urdf (robot description, URDF)
Before this commit: robot amiga_min, 2 links, 1 joints
Joints:
- joint base_to_velodyne: origin xyz=0.0 0.0 0.80 rpy=0 0 0 -> xyz=1.130 0.0 0.80 rpy=0 0 0
